File: d1_mini_clock.sch (KiCad schematic (older format))
At the start: 13 parts, among them J1 Conn_01x04, J2 Conn_01x03, P1 CONN_01X08, P2 CONN_01X08, U1 DS3231M, U2 74AHCT1G125

Commit message: Library updates
Parts:
- J1: symbol conn:Conn_01x04 -> d1_mini_clock-rescue:Conn_01x04-conn
- J2: symbol conn:Conn_01x03 -> d1_mini_clock-rescue:Conn_01x03-conn
Changed lines of the file:
@@
 $EndComp
 $Comp
-L conn:Conn_01x04 J1
+L d1_mini_clock-rescue:Conn_01x04-conn J1
 U 1 1 5FFB79C6
 P 7000 4000
@@
 $EndComp
 $Comp
-L conn:Conn_01x03 J2
+L d1_mini_clock-rescue:Conn_01x03-conn J2
 U 1 1 5FFB808A
 P 7000 4800
